Commit message: Use primitive forearm visuals and extended gripper bodies

File: isaac_lab_data_collection/src/my_robot_description/urdf/biped_s40.urdf (robot description, URDF)
Before this commit: robot my_robot_description, 46 links, 45 joints
Links:
- added link zarm_l_gripper_finger_left, mass 0.01; collision box size=0.01 0.06 0.025; visual box size=0.01 0.06 0.025
- added link zarm_l_gripper_finger_right, mass 0.01; collision box size=0.01 0.06 0.025; visual box size=0.01 0.06 0.025
- added link zarm_r_gripper_finger_left, mass 0.01; collision box size=0.01 0.06 0.025; visual box size=0.01 0.06 0.025
- added link zarm_r_gripper_finger_right, mass 0.01; collision box size=0.01 0.06 0.025; visual box size=0.01 0.06 0.025
- link base_link: geometry visual mesh filename=base_link.STL scale=1 1 1
- link camera: geometry visual mesh filename=camera.STL scale=1 1 1
- link camera_base: geometry collision cylinder length=0.15 radius=0.03; visual mesh filename=camera_base.STL scale=1 1 1
- link leg_l1_link: geometry visual mesh filename=l_leg_yaw.STL scale=1 1 1
- link leg_l2_link: geometry visual mesh filename=l_leg_roll.STL scale=1 1 1
- link leg_l3_link: geometry visual mesh filename=l_leg_pitch.STL scale=1 1 1
- link leg_l4_link: geometry visual mesh filename=l_knee.STL scale=1 1 1
- link leg_l5_link: geometry visual mesh filename=l_foot_pitch.STL scale=1 1 1
- link leg_l6_link: geometry visual mesh filename=l_foot_roll.STL scale=1 1 1
- link leg_r1_link: geometry visual mesh filename=r_leg_yaw.STL scale=1 1 1
- link leg_r2_link: geometry visual mesh filename=r_leg_roll.STL scale=1 1 1
- link leg_r3_link: geometry visual mesh filename=r_leg_pitch.STL scale=1 1 1
- link leg_r4_link: geometry visual mesh filename=r_knee.STL scale=1 1 1
- link leg_r5_link: geometry visual mesh filename=r_foot_pitch.STL scale=1 1 1
- link leg_r6_link: geometry visual mesh filename=r_foot_roll.STL scale=1 1 1
- link zarm_l1_link: geometry visual mesh filename=l_arm_yaw.STL scale=1 1 1
- link zarm_l2_link: geometry visual mesh filename=l_arm_roll.STL scale=1 1 1
- link zarm_l3_link: geometry visual mesh filename=l_arm_pitch.STL scale=1 1 1
- link zarm_l4_link: geometry visual mesh filename=l_forearm.STL scale=1 1 1
- link zarm_l5_link: geometry visual mesh filename=l_hand_pitch.STL scale=1 1 1
- link zarm_l6_link: geometry visual mesh filename=l_hand_roll.STL scale=1 1 1
- link zarm_l7_end_effector: mass None -> 0.05; geometry collision box size=0.05 0.08 0.12; visual box size=0.05 0.08 0.12
- link zarm_l7_link: geometry collision cylinder length=0.14 radius=0.025; visual cylinder length=0.14 radius=0.025
- link zarm_r1_link: geometry visual mesh filename=r_arm_yaw.STL scale=1 1 1
- link zarm_r2_link: geometry visual mesh filename=r_arm_roll.STL scale=1 1 1
- link zarm_r3_link: geometry visual mesh filename=r_arm_pitch.STL scale=1 1 1
- link zarm_r4_link: geometry visual mesh filename=r_forearm.STL scale=1 1 1
- link zarm_r5_link: geometry visual mesh filename=r_hand_pitch.STL scale=1 1 1
- link zarm_r6_link: geometry visual mesh filename=r_hand_roll.STL scale=1 1 1
- link zarm_r7_end_effector: mass None -> 0.05; geometry collision box size=0.05 0.08 0.12; visual box size=0.05 0.08 0.12
- link zarm_r7_link: geometry collision cylinder length=0.14 radius=0.025; visual cylinder length=0.14 radius=0.025
- link zhead_1_link: geometry visual mesh filename=head_yaw.STL scale=1 1 1
- link zhead_2_link: geometry visual mesh filename=head_pitch.STL scale=1 1 1
Joints:
- added joint zarm_l_gripper_finger_left_joint: type prismatic, parent zarm_l7_end_effector, child zarm_l_gripper_finger_left, origin xyz=0 0 0 rpy=0 0 0, axis 0 1 0, limit lower=0 upper=0.035 effort=5 velocity=0.5
- added joint zarm_l_gripper_finger_right_joint: type prismatic, parent zarm_l7_end_effector, child zarm_l_gripper_finger_right, origin xyz=0 0 0 rpy=0 0 0, axis 0 -1 0, limit lower=-0.035 upper=0 effort=5 velocity=0.5, mimic joint=zarm_l_gripper_finger_left_joint multiplier=-1 offset=0
- added joint zarm_r_gripper_finger_left_joint: type prismatic, parent zarm_r7_end_effector, child zarm_r_gripper_finger_left, origin xyz=0 0 0 rpy=0 0 0, axis 0 1 0, limit lower=0 upper=0.035 effort=5 velocity=0.5
- added joint zarm_r_gripper_finger_right_joint: type prismatic, parent zarm_r7_end_effector, child zarm_r_gripper_finger_right, origin xyz=0 0 0 rpy=0 0 0, axis 0 -1 0, limit lower=-0.035 upper=0 effort=5 velocity=0.5, mimic joint=zarm_r_gripper_finger_left_joint multiplier=-1 offset=0
